File: PCB/Spacecraft ATmega328 MOSFET/Spacecraft ATmega328 MOSFET.kicad_pcb (KiCad board)
At the start: 2 copper layers, 38.6 x 31 mm, 34 parts, among them J1 I2C/Power_IN, J2 I2C/Power_IN, J3 Bootloader Pins, J4 LED, J5 SOL_1, SW1 SW_Push, U2 DMN4026SSD, Y1 Crystal

Commit message: Finished Tracing
Parts:
- moved C1 15.5 mm to (105.7, 67.4), turned to 45 degrees
- moved C2 14.1 mm to (114.8, 77.1), turned to 45 degrees
- moved R7 3.82 mm to (101.3, 69.1), turned to 45 degrees
- moved R3 3.50 mm to (104.0, 76.8)
- moved R2 2.34 mm to (101.3, 76.8)
- moved C3 2.24 mm to (103.2, 69.9), turned to 45 degrees
- moved R8 1.94 mm to (103.9, 66.5), turned to 45 degrees
- moved C4 1.83 mm to (100.5, 72.8), turned to 90 degrees
- moved 5V 1.53 mm to (108.0, 62.4), turned to 0 degrees
- moved R5 1.48 mm to (115.1, 63.9), turned to -45 degrees
- moved SW1 1.47 mm to (119.3, 70.2)
- moved C5 1.37 mm to (112.7, 81.1), turned to -90 degrees
- moved C6 1.30 mm to (113.4, 65.6), turned to -45 degrees
- moved R6 1.27 mm to (108.2, 64.9), turned to 45 degrees
- moved Rx 1.15 mm to (104.2, 62.4), turned to 0 degrees
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Routing:
- net GND: track 0.00 -> 103.7 mm, vias 0 -> 10
- net +5V: track 0.00 -> 73.7 mm, vias 0 -> 1
- net VCC: track 0.00 -> 63.1 mm, vias 0 -> 1
- net /SCL: track 0.00 -> 48.6 mm, vias 0 -> 1
- net /SDA: track 0.00 -> 45.5 mm, vias 0 -> 1
- net /SCK: track 0.00 -> 41.0 mm, vias 0 -> 1
- net /Reset: track 0.00 -> 38.4 mm, vias 0 -> 1
- net /MISO: track 0.00 -> 31.3 mm, vias 0 -> 1
- net /MOSI: track 0.00 -> 24.8 mm, vias 0 -> 1
- net /SOL2: track 0.00 -> 21.2 mm
- net /LED: track 0.00 -> 19.3 mm, vias 0 -> 1
- net /TXD: track 0.00 -> 16.6 mm, vias 0 -> 2
- net /Gate1: track 0.00 -> 15.9 mm
- net /RXD: track 0.00 -> 12.7 mm, vias 0 -> 2
- net Net-(C3-Pad2): track 0.00 -> 12.7 mm
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- added copper zone on B.Cu, net GND
Other:
- net class Default removed
- board text added: "Engineering Physics Propulsion Lab Designed by: Dylan Ballback 04/29/22"
- board text removed: "4/25/22"
- board text removed: "Dylan Ballback"
- board text removed: "EPPL"
- board text removed: "Engineering Physics Propulsion Lab"
- board text removed: "V2"
