File: PCB/Pi_HAT/V1/Pi_HAT.kicad_pcb (KiCad board)
At the start: 2 copper layers, 59 x 69.6 mm, 18 parts, among them J1 MPU9250, J2 Pi GPIO, J3 Display, J4 Solenoid I2C, J5 XT60PW-M

Commit message: Added Extra I2C Header
Parts:
- added J6: Solenoid I2C, Connector_PinHeader_2.54mm:PinHeader_1x04_P2.54mm_Vertical, F.Cu at (103.2, 107.3)
- J2: value Pi GPIO -> Pi_GPIO
- TB1: value ARDUINO NANO -> ARDUINO_NANO
- moved G*** 3.58 mm to (142.2, 92.9), turned to 75 degrees
Connections:
- J4 pad 3: /SDA -> /SCL
- J4 pad 4: /SCL -> /SDA
Routing:
- net /SDA: track 66.4 -> 88.8 mm
- net 12V: track 99.9 -> 119.1 mm
- net /SCL: track 68.3 -> 80.9 mm
- net GND: track 88.5 -> 99.9 mm
