File: PCB/NANO_HAT/NANO_HAT/NANO_HAT.kicad_sch (KiCad schematic)
At the start: 18 parts, among them J1 Conn_01x03_Male, J2 Conn_01x02_Male, J3 Conn_01x02_Male, J4 Conn_01x04_Male, J5 Conn_01x02_Male, J6 Conn_01x02_Male, J7 Conn_01x04_Male, U1 DMN4026SSD

Commit message: Updated (Gerber)
Changed lines of the file:
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@@
 (kicad_sch (version 20211123) (generator eeschema)
   (paper "A4")
+  (junction (at 73.66 34.29) (diameter 0) (color 0 0 0 0)
+  )
+  (junction (at 68.58 77.47) (diameter 0) (color 0 0 0 0)
+  )
+  (junction (at 130.81 71.12) (diameter 0) (color 0 0 0 0)
+  )
+  (junction (at 68.58 73.66) (diameter 0) (color 0 0 0 0)
+  )
+  (junction (at 149.86 74.93) (diameter 0) (color 0 0 0 0)
+  )
   (junction (at 109.22 39.37) (diameter 0) (color 0 0 0 0)
   )
-  (junction (at 68.58 77.47) (diameter 0) (color 0 0 0 0)
-  )
-  (junction (at 130.81 71.12) (diameter 0) (color 0 0 0 0)
-  )
-  (junction (at 68.58 73.66) (diameter 0) (color 0 0 0 0)
-  )
-  (junction (at 149.86 74.93) (diameter 0) (color 0 0 0 0)
-  )
   (junction (at 68.58 74.93) (diameter 0) (color 0 0 0 0)
-  )
-  (junction (at 109.22 102.87) (diameter 0) (color 0 0 0 0)
-  )
-  (junction (at 73.66 34.29) (diameter 0) (color 0 0 0 0)
   )
   (junction (at 130.81 78.74) (diameter 0) (color 0 0 0 0)
@@
     (stroke (width 0) (type default) (color 0 0 0 0))
   )
-  (wire (pts (xy 109.22 101.6) (xy 109.22 102.87))
-    (stroke (width 0) (type default) (color 0 0 0 0))
-  )
   (wire (pts (xy 68.58 73.66) (xy 78.74 73.66))
     (stroke (width 0) (type default) (color 0 0 0 0))
@@
     (pin "3")
     (pin "4")
-  )
-  (symbol (lib_id "HPS:PWR_FLAG") (at 73.66 34.29 0) (unit 1)
-    (in_bom yes) (on_board yes) (fields_autoplaced)
-    (property "Reference" "#FLG0102" (id 0) (at 73.66 32.385 0)
-      (effects (font (size 1.27 1.27)) hide)
-    )
-    (property "Value" "PWR_FLAG" (id 1) (at 73.66 29.21 0))
-    (property "Footprint" "" (id 2) (at 73.66 34.29 0)
-      (effects (font (size 1.27 1.27)) hide)
-    )
-    (property "Datasheet" "~" (id 3) (at 73.66 34.29 0)
-      (effects (font (size 1.27 1.27)) hide)
-    )
-    (pin "1")
   )
   (symbol (lib_id "HPS:MountingHole") (at 234.95 25.4 0) (unit 1)
@@
     (pin "2")
   )
-  (symbol (lib_id "HPS:PWR_FLAG") (at 109.22 101.6 0) (unit 1)
-    (in_bom yes) (on_board yes) (fields_autoplaced)
-    (property "Reference" "#FLG0103" (id 0) (at 109.22 99.695 0)
-      (effects (font (size 1.27 1.27)) hide)
-    )
-    (property "Value" "PWR_FLAG" (id 1) (at 109.22 96.52 0))
-    (property "Footprint" "" (id 2) (at 109.22 101.6 0)
-      (effects (font (size 1.27 1.27)) hide)
-    )
-    (property "Datasheet" "~" (id 3) (at 109.22 101.6 0)
+  (symbol (lib_id "power:PWR_FLAG") (at 73.66 34.29 0) (unit 1)
+    (in_bom yes) (on_board yes) (fields_autoplaced)
+    (property "Reference" "#FLG0101" (id 0) (at 73.66 32.385 0)
+      (effects (font (size 1.27 1.27)) hide)
+    )
+    (property "Value" "" (id 1) (at 73.66 28.8036 0))
+    (property "Footprint" "" (id 2) (at 73.66 34.29 0)
+      (effects (font (size 1.27 1.27)) hide)
+    )
+    (property "Datasheet" "~" (id 3) (at 73.66 34.29 0)
       (effects (font (size 1.27 1.27)) hide)
     )
@@
     )
     (property "Datasheet" "" (id 3) (at 109.22 39.37 0)
-      (effects (font (size 1.27 1.27)) hide)
-    )
-    (pin "1")
-  )
-  (symbol (lib_id "HPS:PWR_FLAG") (at 109.22 39.37 180) (unit 1)
-    (in_bom yes) (on_board yes) (fields_autoplaced)
-    (property "Reference" "#FLG0101" (id 0) (at 109.22 41.275 0)
-      (effects (font (size 1.27 1.27)) hide)
-    )
-    (property "Value" "PWR_FLAG" (id 1) (at 109.22 44.45 0))
-    (property "Footprint" "" (id 2) (at 109.22 39.37 0)
-      (effects (font (size 1.27 1.27)) hide)
-    )
-    (property "Datasheet" "~" (id 3) (at 109.22 39.37 0)
       (effects (font (size 1.27 1.27)) hide)
     )
@@
     (pin "1")
   )
+  (symbol (lib_id "power:PWR_FLAG") (at 109.22 39.37 0) (unit 1)
+    (in_bom yes) (on_board yes) (fields_autoplaced)
+    (property "Reference" "#FLG0102" (id 0) (at 109.22 37.465 0)
+      (effects (font (size 1.27 1.27)) hide)
+    )
+    (property "Value" "PWR_FLAG" (id 1) (at 109.22 33.8836 0))
+    (property "Footprint" "" (id 2) (at 109.22 39.37 0)
+      (effects (font (size 1.27 1.27)) hide)
+    )
+    (property "Datasheet" "~" (id 3) (at 109.22 39.37 0)
+      (effects (font (size 1.27 1.27)) hide)
+    )
+    (pin "1")
+  )
   (sheet_instances
     (path "/" (page "1"))
   )
   (symbol_instances
-    (path "/b9bb5d52-b7d5-43ed-8430-3e0ce9f739f2"
+    (path "/379134a3-e40e-433e-8b90-c39a8d291532"
       (reference "#FLG0101") (unit 1) (value "PWR_FLAG") (footprint "")
     )
-    (path "/22d6bc29-553d-4594-853b-612f0e90127b"
+    (path "/f7b4f25e-9991-4695-897f-d29298d9dbc3"
       (reference "#FLG0102") (unit 1) (value "PWR_FLAG") (footprint "")
     )
-    (path "/3343345a-4a1e-479e-97fe-80c94fd5ca3a"
-      (reference "#FLG0103") (unit 1) (value "PWR_FLAG") (footprint "")
-    )
     (path "/92d90d55-662a-48fe-b9fb-40a32d8e5125"
