File: PCB/NANO_HAT/NANO_HAT/NANO_HAT.kicad_pcb (KiCad board)
At the start: 2 copper layers, 18 parts, among them J1 Conn_01x03_Male, J2 Conn_01x02_Male, J3 Conn_01x02_Male, J4 Conn_01x04_Male, J5 Conn_01x02_Male, J6 Conn_01x02_Male, J7 Conn_01x04_Male, U1 DMN4026SSD

Commit message: NANO_HAT Update 2
Routing:
- net /SOL1: track 29.4 -> 64.8 mm
- net /SOL2: track 30.6 -> 43.7 mm
- net VCC: track 143.3 -> 149.8 mm
- added copper zone on B.Cu, net GND
Other:
- board outline added: 54 x 60.2 mm
