File: PCB/CubeSat/CubeSat.kicad_pcb (KiCad board)
At the start: 2 copper layers, 88 x 73 mm, 11 parts, among them J1 Li 24V Battery, J2 MPU 6050, J3 Conn_01x08, J4 Conn_02x20_Odd_Even, U1 LM2596S

Commit message: Finished/Uploaded Gerber
Parts:
- moved H5 50.7 mm to (113.0, 110.6)
- moved H6 12.5 mm to (113.0, 52.4)
- moved J3 1.70 mm to (130.3, 49.9)
- moved J4 1.60 mm to (111.8, 57.4)
Routing:
- net VCC: track 0.00 -> 118.7 mm
- net /CHA: track 0.00 -> 95.6 mm
- net /CHB: track 0.00 -> 89.4 mm
- net /CW/CCW: track 0.00 -> 80.6 mm
- net /PWM: track 0.00 -> 79.1 mm
- net /brake: track 0.00 -> 70.7 mm
- net /SDA: track 0.00 -> 59.6 mm, vias 0 -> 1
- net /SCL: track 0.00 -> 58.0 mm, vias 0 -> 1
- net /5VB: track 0.00 -> 55.4 mm
- net /3.3V: track 0.00 -> 50.3 mm
- added copper zone on F.Cu, net GND
