File: ISAAC/PCB/NANO_HAT/NANO_HAT/NANO_HAT.kicad_sch (KiCad schematic)
At the start: 18 parts, among them J1 Conn_01x03_Male, J2 Conn_01x02_Male, J3 Conn_01x02_Male, J4 Conn_01x04_Male, J5 Conn_01x02_Male, J6 Conn_01x02_Male, J7 Conn_01x04_Male, U1 DMN4026SSD

Commit message: Fixed NANO_HAT
Parts:
- added C1: 0.33 uF, symbol Device:C
- added C2: 0.1uF, Capacitor_SMD:C_0603_1608Metric_Pad1.08x0.95mm_HandSolder, symbol Device:C_Polarized_US
Connections:
- net 5V: now also C2.1
- net GND: now also C1.2, C2.2
- net VCC: now also C1.1
Changed lines of the file:
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@@
   (junction (at 130.81 71.12) (diameter 0) (color 0 0 0 0)
+  )
+  (junction (at 109.22 44.069) (diameter 0) (color 0 0 0 0)
   )
   (junction (at 68.58 73.66) (diameter 0) (color 0 0 0 0)
@@
     (stroke (width 0) (type default) (color 0 0 0 0))
   )
+  (wire (pts (xy 73.66 41.91) (xy 73.66 44.069))
+    (stroke (width 0) (type default) (color 0 0 0 0))
+  )
   (wire (pts (xy 144.78 71.12) (xy 149.86 71.12))
     (stroke (width 0) (type default) (color 0 0 0 0))
   )
+  (wire (pts (xy 109.22 39.37) (xy 109.22 44.069))
+    (stroke (width 0) (type default) (color 0 0 0 0))
+  )
   (wire (pts (xy 109.22 105.41) (xy 111.76 105.41))
     (stroke (width 0) (type default) (color 0 0 0 0))
@@
     (stroke (width 0) (type default) (color 0 0 0 0))
   )
-  (wire (pts (xy 109.22 34.29) (xy 114.3 34.29))
+  (wire (pts (xy 109.22 34.29) (xy 119.38 34.29))
     (stroke (width 0) (type default) (color 0 0 0 0))
   )
@@
     (stroke (width 0) (type default) (color 0 0 0 0))
   )
+  (wire (pts (xy 73.66 44.069) (xy 109.22 44.069))
+    (stroke (width 0) (type default) (color 0 0 0 0))
+  )
   (wire (pts (xy 149.86 74.93) (xy 153.67 74.93))
+    (stroke (width 0) (type default) (color 0 0 0 0))
+  )
+  (wire (pts (xy 119.38 36.449) (xy 119.38 34.29))
+    (stroke (width 0) (type default) (color 0 0 0 0))
+  )
+  (wire (pts (xy 109.22 44.069) (xy 119.38 44.069))
     (stroke (width 0) (type default) (color 0 0 0 0))
   )
@@
       (effects (font (size 1.27 1.27)) hide)
     )
-    (property "Value" "" (id 1) (at 73.66 28.8036 0))
+    (property "Value" "PWR_FLAG" (id 1) (at 73.66 28.8036 0))
     (property "Footprint" "" (id 2) (at 73.66 34.29 0)
       (effects (font (size 1.27 1.27)) hide)
@@
     (pin "1")
   )
+  (symbol (lib_id "Device:C_Polarized_US") (at 119.38 40.259 0) (unit 1)
+    (in_bom yes) (on_board yes) (fields_autoplaced)
+    (property "Reference" "C2" (id 0) (at 123.19 38.3539 0)
+      (effects (font (size 1.27 1.27)) (justify left))
+    )
+    (property "Value" "0.1uF" (id 1) (at 123.19 40.8939 0)
+      (effects (font (size 1.27 1.27)) (justify left))
+    )
+    (property "Footprint" "Capacitor_SMD:C_0603_1608Metric_Pad1.08x0.95mm_HandSolder" (id 2) (at 119.38 40.259 0)
+      (effects (font (size 1.27 1.27)) hide)
+    )
+    (property "Datasheet" "~" (id 3) (at 119.38 40.259 0)
+      (effects (font (size 1.27 1.27)) hide)
+    )
+    (pin "1")
+    (pin "2")
+  )
   (symbol (lib_id "Connector:Conn_01x04_Male") (at 130.81 104.14 0) (unit 1)
     (in_bom yes) (on_board yes) (fields_autoplaced)
@@
       (effects (font (size 1.27 1.27)) hide)
     )
+  )
+  (symbol (lib_id "Device:C") (at 73.66 38.1 0) (unit 1)
+    (in_bom yes) (on_board yes)
+    (property "Reference" "C1" (id 0) (at 74.549 35.941 0)
+      (effects (font (size 1.27 1.27)) (justify left))
+    )
+    (property "Value" "0.33 uF" (id 1) (at 64.008 40.005 0)
+      (effects (font (size 1.27 1.27)) (justify left))
+    )
+    (property "Footprint" "" (id 2) (at 74.6252 41.91 0)
+      (effects (font (size 1.27 1.27)) hide)
+    )
+    (property "Datasheet" "~" (id 3) (at 73.66 38.1 0)
+      (effects (font (size 1.27 1.27)) hide)
+    )
+    (pin "1")
+    (pin "2")
   )
   (symbol (lib_id "HPS:GND") (at 227.33 138.43 90) (unit 1)
@@
       (reference "#PWR0115") (unit 1) (value "GND") (footprint "")
     )
+    (path "/6e72ccaa-c091-4330-a23e-92e3f7e9d19d"
+      (reference "C1") (unit 1) (value "0.33 uF") (footprint "Capacitor_SMD:C_0603_1608Metric_Pad1.08x0.95mm_HandSolder")
+    )
+    (path "/43d3000c-741a-401c-86de-e704c20a31b7"
+      (reference "C2") (unit 1) (value "0.1uF") (footprint "Capacitor_SMD:C_0603_1608Metric_Pad1.08x0.95mm_HandSolder")
+    )
     (path "/855d7662-117e-44c7-bac9-dc6937631075"
