File: Cubesat/PCB/CubeSat/CubeSat.kicad_pcb (KiCad board)
At the start: 2 copper layers, 88 x 73 mm, 11 parts, among them J1 Li 24V Battery, J2 MPU 6050, J3 Conn_01x08, J4 Conn_02x20_Odd_Even, U1 LM2596S

Commit message: Fixed PCB
Parts:
- moved J3 17.8 mm to (148.1, 49.9), turned to -90 degrees
Connections:
- J4 pad 4: unconnected-(J4-Pad4) -> /5VB
- J4 pad 6: unconnected-(J4-Pad6) -> GND
Routing:
- net /CHA: track 95.6 -> 72.4 mm
- net VCC: track 118.7 -> 124.1 mm
- net /CHB: track 89.4 -> 84.9 mm
- net /brake: track 70.7 -> 75.1 mm
- net /5VB: track 55.4 -> 58.0 mm
- net /CW/CCW: track 80.6 -> 81.5 mm
