File: Cubesat/PCB/CubeSat/CubeSat.kicad_sch (KiCad schematic)
At the start: 11 parts, among them J1 Li 24V Battery, J2 MPU 6050, J3 Conn_01x08, J4 Conn_02x20_Odd_Even, U1 LM2596S

Commit message: Fixed PCB
Connections:
- net 5VB: now also J4.4 (Pin_4)
- net GND: now also J4.6 (Pin_6)
- no-connect marks 34 -> 32
Changed lines of the file:
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@@
   (no_connect (at 180.34 72.39))
   (no_connect (at 180.34 69.85))
-  (no_connect (at 180.34 67.31))
-  (no_connect (at 180.34 64.77))
   (no_connect (at 167.64 82.55))
   (no_connect (at 167.64 85.09))
@@
     (stroke (width 0) (type default) (color 0 0 0 0))
   )
+  (wire (pts (xy 186.69 64.77) (xy 180.34 64.77))
+    (stroke (width 0) (type default) (color 0 0 0 0))
+  )
   (wire (pts (xy 114.3 92.71) (xy 120.65 92.71))
     (stroke (width 0) (type default) (color 0 0 0 0))
@@
   (label "brake" (at 161.29 97.79 0)
     (effects (font (size 1.27 1.27)) (justify left bottom))
+  )
+  (label "5VB" (at 186.69 64.77 180)
+    (effects (font (size 1.27 1.27)) (justify right bottom))
   )
   (label "3.3V" (at 114.3 62.23 0)
@@
     (pin "3")
     (pin "4")
+  )
+  (symbol (lib_id "power:GND") (at 180.34 67.31 90) (unit 1)
+    (in_bom yes) (on_board yes) (fields_autoplaced)
+    (property "Reference" "#PWR?" (id 0) (at 186.69 67.31 0)
+      (effects (font (size 1.27 1.27)) hide)
+    )
+    (property "Value" "GND" (id 1) (at 184.15 67.3099 90)
+      (effects (font (size 1.27 1.27)) (justify right))
+    )
+    (property "Footprint" "" (id 2) (at 180.34 67.31 0)
+      (effects (font (size 1.27 1.27)) hide)
+    )
+    (property "Datasheet" "" (id 3) (at 180.34 67.31 0)
+      (effects (font (size 1.27 1.27)) hide)
+    )
+    (pin "1")
   )
   (symbol (lib_id "Mechanical:MountingHole") (at 121.92 40.64 0) (unit 1)
@@
       (reference "#PWR0106") (unit 1) (value "GND") (footprint "")
     )
+    (path "/624f9c04-0a3b-4bde-9c91-899219f49d93"
+      (reference "#PWR?") (unit 1) (value "GND") (footprint "")
+    )
     (path "/c125495c-82f3-42db-8b42-bf22cefa9f79"
