File: ISAAC/PCB/Free_Flier_PCB/Free_Flier_PCB.kicad_pcb (KiCad board)
At the start: 2 copper layers, 40.9 x 28.7 mm, 21 parts, among them J1 Power and Data Female, J2 LED Female, J3 Solenoid Conn, J4 Programming Pins Female, SW1 SW_Push_Dual, U1 ATmega328P-AU, U2 DMN4026SSD, U3 LM78M05CDTX/NOPB, Y1 16MHz

Commit message: Updated ISAAC & CubeSat
Created Pi HAT V3 PCB and new CubeSat PCB
Connections:
- C5 pad 2: Net-(C5-Pad2) -> unconnected-(U1-Pad7)
- C6 pad 2: Net-(C6-Pad2) -> unconnected-(U1-Pad8)
- R1 pad 2: Net-(R1-Pad2) -> unconnected-(U1-Pad29)
- U1 pad 1: Net-(U1-Pad1) -> unconnected-(U1-Pad1)
- U1 pad 12: Net-(U1-Pad12) -> unconnected-(U1-Pad12)
- U1 pad 13: Net-(U1-Pad13) -> unconnected-(U1-Pad13)
- U1 pad 14: Net-(U1-Pad14) -> unconnected-(U1-Pad14)
- U1 pad 15: Net-(U1-Pad15) -> unconnected-(U1-Pad15)
- U1 pad 16: Net-(U1-Pad16) -> unconnected-(U1-Pad16)
- U1 pad 17: Net-(U1-Pad17) -> unconnected-(U1-Pad17)
- U1 pad 19: Net-(U1-Pad19) -> unconnected-(U1-Pad19)
- U1 pad 2: Net-(U1-Pad2) -> unconnected-(U1-Pad2)
- U1 pad 22: Net-(U1-Pad22) -> unconnected-(U1-Pad22)
- U1 pad 23: Net-(U1-Pad23) -> unconnected-(U1-Pad23)
- U1 pad 24: Net-(U1-Pad24) -> unconnected-(U1-Pad24)
- U1 pad 25: Net-(U1-Pad25) -> unconnected-(U1-Pad25)
- U1 pad 26: Net-(U1-Pad26) -> unconnected-(U1-Pad26)
- U1 pad 29: Net-(R1-Pad2) -> unconnected-(U1-Pad29)
- U1 pad 32: Net-(U1-Pad32) -> unconnected-(U1-Pad32)
- U1 pad 7: Net-(C5-Pad2) -> unconnected-(U1-Pad7)
- U1 pad 8: Net-(C6-Pad2) -> unconnected-(U1-Pad8)
- Y1 pad 1: Net-(C5-Pad2) -> unconnected-(U1-Pad7)
- Y1 pad 2: Net-(C6-Pad2) -> unconnected-(U1-Pad8)
Other:
- net class Default removed
