File: Cubesat/PCB/MJBOTS-CubeSat/A-D Converter.kicad_sch (KiCad schematic)
At the start: 2 parts, among them J11 JST-BATT, U2 MCP3008-I/SL

Commit message: Final Updates "HOPEFULLY"
Parts:
- removed J11: JST-BATT, Connector_PinHeader_2.54mm:PinHeader_1x04_P2.54mm_Vertical, symbol 24V_Li_batt:Conn_01x04
- added R1: 2k, Resistor_SMD:R_0805_2012Metric_Pad1.20x1.40mm_HandSolder, symbol Device:R_US
- added R2: 1k, Resistor_SMD:R_0805_2012Metric_Pad1.20x1.40mm_HandSolder, symbol Device:R_US
Connections:
- net GND: now also R2.2
- net CELL1 renamed 12V
- net 12V: now also R1.1, R2.1
- net CELL2: no longer names the net of U2.2 (CH1)
- net CELL3: no longer names the net of U2.3 (CH2)
- net VT: no longer names the net of U2.4 (CH3)
- new net VCC: R1.2
- no-connect marks 4 -> 7
Changed lines of the file:
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@@
   (junction (at 159.512 75.692) (diameter 0) (color 0 0 0 0)
+  )
+  (junction (at 92.71 86.868) (diameter 0) (color 0 0 0 0)
   )
   (no_connect (at 123.952 96.012))
@@
   (no_connect (at 123.952 101.092))
   (no_connect (at 123.952 93.472))
-  (wire (pts (xy 183.134 93.98) (xy 188.976 93.98))
-    (stroke (width 0) (type default) (color 0 0 0 0))
-  )
+  (no_connect (at 123.952 88.392))
+  (no_connect (at 123.952 90.932))
+  (no_connect (at 123.952 85.852))
   (wire (pts (xy 120.396 80.772) (xy 123.952 80.772))
     (stroke (width 0) (type default) (color 0 0 0 0))
   )
-  (wire (pts (xy 118.11 90.932) (xy 123.952 90.932))
-    (stroke (width 0) (type default) (color 0 0 0 0))
-  )
-  (wire (pts (xy 118.11 88.392) (xy 123.952 88.392))
+  (wire (pts (xy 120.396 83.312) (xy 123.952 83.312))
     (stroke (width 0) (type default) (color 0 0 0 0))
   )
   (wire (pts (xy 119.634 106.172) (xy 123.952 106.172))
-    (stroke (width 0) (type default) (color 0 0 0 0))
-  )
-  (wire (pts (xy 183.134 101.6) (xy 188.976 101.6))
     (stroke (width 0) (type default) (color 0 0 0 0))
   )
@@
     (stroke (width 0) (type default) (color 0 0 0 0))
   )
-  (wire (pts (xy 118.11 83.312) (xy 123.952 83.312))
-    (stroke (width 0) (type default) (color 0 0 0 0))
-  )
-  (wire (pts (xy 183.134 99.06) (xy 188.976 99.06))
-    (stroke (width 0) (type default) (color 0 0 0 0))
-  )
-  (wire (pts (xy 118.11 85.852) (xy 123.952 85.852))
-    (stroke (width 0) (type default) (color 0 0 0 0))
-  )
   (wire (pts (xy 119.634 103.632) (xy 123.952 103.632))
-    (stroke (width 0) (type default) (color 0 0 0 0))
-  )
-  (wire (pts (xy 183.134 96.52) (xy 188.976 96.52))
     (stroke (width 0) (type default) (color 0 0 0 0))
   )
@@
     (stroke (width 0) (type default) (color 0 0 0 0))
   )
-  (label "VT" (at 118.11 90.932 0)
+  (wire (pts (xy 92.71 86.868) (xy 96.52 86.868))
+    (stroke (width 0) (type default) (color 0 0 0 0))
+  )
+  (label "12V" (at 120.396 83.312 0)
     (effects (font (size 1.27 1.27)) (justify left bottom))
   )
-  (label "CELL2" (at 118.11 85.852 0)
-    (effects (font (size 1.27 1.27)) (justify left bottom))
-  )
-  (label "CELL1" (at 183.134 93.98 0)
-    (effects (font (size 1.27 1.27)) (justify left bottom))
-  )
-  (label "CELL3" (at 183.134 99.06 0)
-    (effects (font (size 1.27 1.27)) (justify left bottom))
-  )
-  (label "CELL2" (at 183.134 96.52 0)
-    (effects (font (size 1.27 1.27)) (justify left bottom))
-  )
-  (label "CELL3" (at 118.11 88.392 0)
-    (effects (font (size 1.27 1.27)) (justify left bottom))
-  )
-  (label "VT" (at 183.134 101.6 0)
-    (effects (font (size 1.27 1.27)) (justify left bottom))
-  )
-  (label "CELL1" (at 118.11 83.312 0)
-    (effects (font (size 1.27 1.27)) (justify left bottom))
+  (label "12V" (at 96.52 86.868 180)
+    (effects (font (size 1.27 1.27)) (justify right bottom))
   )
   (hierarchical_label "MISO" (shape input) (at 163.83 80.772 0)
@@
   (hierarchical_label "3.3V" (shape input) (at 163.83 75.692 0)
     (effects (font (size 1.27 1.27)) (justify left))
+  )
+  (hierarchical_label "VCC" (shape input) (at 92.71 79.248 180)
+    (effects (font (size 1.27 1.27)) (justify right))
   )
   (hierarchical_label "SCLK" (shape input) (at 119.634 103.632 180)
@@
     )
     (property "Datasheet" "" (id 3) (at 159.512 118.872 0)
+      (effects (font (size 1.27 1.27)) hide)
+    )
+    (pin "1")
+  )
+  (symbol (lib_id "Device:R_US") (at 92.71 83.058 180) (unit 1)
+    (in_bom yes) (on_board yes) (fields_autoplaced)
+    (property "Reference" "R1" (id 0) (at 95.25 81.7879 0)
+      (effects (font (size 1.27 1.27)) (justify right))
+    )
+    (property "Value" "2k" (id 1) (at 95.25 84.3279 0)
+      (effects (font (size 1.27 1.27)) (justify right))
+    )
+    (property "Footprint" "Resistor_SMD:R_0805_2012Metric_Pad1.20x1.40mm_HandSolder" (id 2) (at 91.694 82.804 90)
+      (effects (font (size 1.27 1.27)) hide)
+    )
+    (property "Datasheet" "https://www.digikey.com/en/products/detail/te-connectivity-passive-product/RA73F2A2K0BTD/16031942" (id 3) (at 92.71 83.058 0)
+      (effects (font (size 1.27 1.27)) hide)
+    )
+    (pin "1")
+    (pin "2")
+  )
+  (symbol (lib_id "power:GND") (at 92.71 94.488 0) (unit 1)
+    (in_bom yes) (on_board yes) (fields_autoplaced)
+    (property "Reference" "#PWR0116" (id 0) (at 92.71 100.838 0)
+      (effects (font (size 1.27 1.27)) hide)
+    )
+    (property "Value" "GND" (id 1) (at 95.504 95.7579 0)
+      (effects (font (size 1.27 1.27)) (justify left))
+    )
+    (property "Footprint" "" (id 2) (at 92.71 94.488 0)
+      (effects (font (size 1.27 1.27)) hide)
+    )
+    (property "Datasheet" "" (id 3) (at 92.71 94.488 0)
       (effects (font (size 1.27 1.27)) hide)
     )
@@
     (pin "1")
   )
-  (symbol (lib_id "24V_Li_batt:Conn_01x04") (at 194.056 96.52 0) (unit 1)
+  (symbol (lib_id "Device:R_US") (at 92.71 90.678 0) (unit 1)
     (in_bom yes) (on_board yes) (fields_autoplaced)
-    (property "Reference" "J11" (id 0) (at 196.85 96.5199 0)
+    (property "Reference" "R2" (id 0) (at 95.25 89.4079 0)
       (effects (font (size 1.27 1.27)) (justify left))
     )
-    (property "Value" "JST-BATT" (id 1) (at 196.85 99.0599 0)
+    (property "Value" "1k" (id 1) (at 95.25 91.9479 0)
       (effects (font (size 1.27 1.27)) (justify left))
     )
-    (property "Footprint" "Connector_PinHeader_2.54mm:PinHeader_1x04_P2.54mm_Vertical" (id 2) (at 194.056 96.52 0)
+    (property "Footprint" "Resistor_SMD:R_0805_2012Metric_Pad1.20x1.40mm_HandSolder" (id 2) (at 93.726 90.932 90)
       (effects (font (size 1.27 1.27)) hide)
     )
-    (property "Datasheet" "~" (id 3) (at 194.056 96.52 0)
+    (property "Datasheet" "https://www.digikey.com/en/products/detail/te-connectivity-passive-product/RA73F2A1K0BTD/16031399" (id 3) (at 92.71 90.678 0)
       (effects (font (size 1.27 1.27)) hide)
     )
     (pin "1")
     (pin "2")
-    (pin "3")
-    (pin "4")
   )
 )
