File: ISAAC/PCB/Pi_HAT/V3/Pi_HAT_V3/A-D Converter.kicad_sch (KiCad schematic)
At the start: 1 part, among them U2 MCP3008-I/SL

Commit message: Shit ton of stuf
Parts:
- added J9: JST-BATT, Connector_PinHeader_2.54mm:PinHeader_1x04_P2.54mm_Vertical, symbol 24V_Li_batt:Conn_01x04
Connections:
- net CELL1: now reaches U2.2 (CH1)
- net CELL1: now also J9.1 (Pin_1)
- net CELL2: now reaches U2.3 (CH2)
- net CELL2: now also J9.2 (Pin_2)
- net CELL3: now reaches U2.4 (CH3)
- net CELL3: now also J9.3 (Pin_3)
- net VT: now reaches U2.5 (CH4)
- net VT: now also J9.4 (Pin_4)
- no-connect marks 7 -> 3
Changed lines of the file:
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@@
   (no_connect (at 125.73 90.932))
   (no_connect (at 125.73 93.472))
-  (no_connect (at 125.73 78.232))
-  (no_connect (at 125.73 80.772))
-  (no_connect (at 125.73 83.312))
-  (no_connect (at 125.73 85.852))
-  (wire (pts (xy 115.57 75.692) (xy 125.73 75.692))
+  (wire (pts (xy 169.418 92.202) (xy 175.26 92.202))
     (stroke (width 0) (type default) (color 0 0 0 0))
   )
@@
     (stroke (width 0) (type default) (color 0 0 0 0))
   )
+  (wire (pts (xy 119.888 78.232) (xy 125.73 78.232))
+    (stroke (width 0) (type default) (color 0 0 0 0))
+  )
+  (wire (pts (xy 169.418 89.662) (xy 175.26 89.662))
+    (stroke (width 0) (type default) (color 0 0 0 0))
+  )
   (wire (pts (xy 125.73 101.092) (xy 121.412 101.092))
     (stroke (width 0) (type default) (color 0 0 0 0))
   )
+  (wire (pts (xy 169.418 87.122) (xy 175.26 87.122))
+    (stroke (width 0) (type default) (color 0 0 0 0))
+  )
+  (wire (pts (xy 119.888 83.312) (xy 125.73 83.312))
+    (stroke (width 0) (type default) (color 0 0 0 0))
+  )
   (wire (pts (xy 122.174 73.152) (xy 125.73 73.152))
+    (stroke (width 0) (type default) (color 0 0 0 0))
+  )
+  (wire (pts (xy 119.888 80.772) (xy 125.73 80.772))
     (stroke (width 0) (type default) (color 0 0 0 0))
   )
@@
   (wire (pts (xy 161.29 68.072) (xy 165.608 68.072))
     (stroke (width 0) (type default) (color 0 0 0 0))
+  )
+  (wire (pts (xy 169.418 84.582) (xy 175.26 84.582))
+    (stroke (width 0) (type default) (color 0 0 0 0))
+  )
+  (wire (pts (xy 119.888 85.852) (xy 125.73 85.852))
+    (stroke (width 0) (type default) (color 0 0 0 0))
+  )
+  (wire (pts (xy 122.174 75.692) (xy 125.73 75.692))
+    (stroke (width 0) (type default) (color 0 0 0 0))
+  )
+  (label "CELL2" (at 169.418 87.122 0)
+    (effects (font (size 1.27 1.27)) (justify left bottom))
+  )
+  (label "CELL1" (at 169.418 84.582 0)
+    (effects (font (size 1.27 1.27)) (justify left bottom))
+  )
+  (label "CELL3" (at 119.888 83.312 0)
+    (effects (font (size 1.27 1.27)) (justify left bottom))
+  )
+  (label "VT" (at 119.888 85.852 0)
+    (effects (font (size 1.27 1.27)) (justify left bottom))
+  )
+  (label "CELL2" (at 119.888 80.772 0)
+    (effects (font (size 1.27 1.27)) (justify left bottom))
+  )
+  (label "CELL3" (at 169.418 89.662 0)
+    (effects (font (size 1.27 1.27)) (justify left bottom))
+  )
+  (label "CELL1" (at 119.888 78.232 0)
+    (effects (font (size 1.27 1.27)) (justify left bottom))
+  )
+  (label "VT" (at 169.418 92.202 0)
+    (effects (font (size 1.27 1.27)) (justify left bottom))
   )
   (hierarchical_label "3.3V" (shape input) (at 121.412 101.092 180)
@@
     (effects (font (size 1.27 1.27)) (justify right))
   )
-  (hierarchical_label "PS" (shape input) (at 115.57 75.692 180)
+  (hierarchical_label "PS" (shape input) (at 122.174 75.692 180)
     (effects (font (size 1.27 1.27)) (justify right))
   )
+  (symbol (lib_id "24V_Li_batt:Conn_01x04") (at 180.34 87.122 0) (unit 1)
+    (in_bom yes) (on_board yes) (fields_autoplaced)
+    (property "Reference" "J9" (id 0) (at 183.134 87.1219 0)
+      (effects (font (size 1.27 1.27)) (justify left))
+    )
+    (property "Value" "JST-BATT" (id 1) (at 183.134 89.6619 0)
+      (effects (font (size 1.27 1.27)) (justify left))
+    )
+    (property "Footprint" "Connector_PinHeader_2.54mm:PinHeader_1x04_P2.54mm_Vertical" (id 2) (at 180.34 87.122 0)
+      (effects (font (size 1.27 1.27)) hide)
+    )
+    (property "Datasheet" "~" (id 3) (at 180.34 87.122 0)
+      (effects (font (size 1.27 1.27)) hide)
+    )
+    (pin "1")
+    (pin "2")
+    (pin "3")
+    (pin "4")
+  )
   (symbol (lib_id "power:GND") (at 161.29 111.252 90) (unit 1)

Commit message: Final Updates "HOPEFULLY"
Parts:
- removed J9: JST-BATT, Connector_PinHeader_2.54mm:PinHeader_1x04_P2.54mm_Vertical, symbol 24V_Li_batt:Conn_01x04
- added R1, R7: 2k, Resistor_SMD:R_0805_2012Metric_Pad1.20x1.40mm_HandSolder, symbol Device:R_US
- added R6, R8: 1k, Resistor_SMD:R_0805_2012Metric_Pad1.20x1.40mm_HandSolder, symbol Device:R_US
Connections:
- net GND: now also R6.2, R8.2
- net CELL1 renamed 4V0
- net 4V0: now also R7.2, R8.1
- net CELL2 renamed 4V1
- net 4V1: now also R1.2, R6.1
- net CELL3: no longer names the net of U2.4 (CH3)
- net VT: no longer names the net of U2.5 (CH4)
- new net VCC0: R7.1
- new net VCC1: R1.1
- no-connect marks 3 -> 5
Changed lines of the file:
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@@
 (kicad_sch (version 20211123) (generator eeschema)
   (paper "A4")
+  (junction (at 94.488 78.994) (diameter 0) (color 0 0 0 0)
+  )
   (junction (at 161.29 68.072) (diameter 0) (color 0 0 0 0)
+  )
+  (junction (at 106.172 78.74) (diameter 0) (color 0 0 0 0)
   )
   (no_connect (at 125.73 88.392))
   (no_connect (at 125.73 90.932))
   (no_connect (at 125.73 93.472))
-  (wire (pts (xy 169.418 92.202) (xy 175.26 92.202))
+  (no_connect (at 125.73 83.312))
+  (no_connect (at 125.73 85.852))
+  (wire (pts (xy 119.888 78.232) (xy 125.73 78.232))
     (stroke (width 0) (type default) (color 0 0 0 0))
   )
@@
     (stroke (width 0) (type default) (color 0 0 0 0))
   )
-  (wire (pts (xy 119.888 78.232) (xy 125.73 78.232))
-    (stroke (width 0) (type default) (color 0 0 0 0))
-  )
-  (wire (pts (xy 169.418 89.662) (xy 175.26 89.662))
-    (stroke (width 0) (type default) (color 0 0 0 0))
-  )
   (wire (pts (xy 125.73 101.092) (xy 121.412 101.092))
     (stroke (width 0) (type default) (color 0 0 0 0))
   )
-  (wire (pts (xy 169.418 87.122) (xy 175.26 87.122))
-    (stroke (width 0) (type default) (color 0 0 0 0))
-  )
-  (wire (pts (xy 119.888 83.312) (xy 125.73 83.312))
+  (wire (pts (xy 119.888 80.772) (xy 125.73 80.772))
     (stroke (width 0) (type default) (color 0 0 0 0))
   )
@@
     (stroke (width 0) (type default) (color 0 0 0 0))
   )
-  (wire (pts (xy 119.888 80.772) (xy 125.73 80.772))
-    (stroke (width 0) (type default) (color 0 0 0 0))
-  )
   (wire (pts (xy 121.412 96.012) (xy 125.73 96.012))
     (stroke (width 0) (type default) (color 0 0 0 0))
   )
+  (wire (pts (xy 106.172 78.74) (xy 111.506 78.74))
+    (stroke (width 0) (type default) (color 0 0 0 0))
+  )
   (wire (pts (xy 161.29 68.072) (xy 165.608 68.072))
     (stroke (width 0) (type default) (color 0 0 0 0))
   )
-  (wire (pts (xy 169.418 84.582) (xy 175.26 84.582))
-    (stroke (width 0) (type default) (color 0 0 0 0))
-  )
-  (wire (pts (xy 119.888 85.852) (xy 125.73 85.852))
-    (stroke (width 0) (type default) (color 0 0 0 0))
-  )
   (wire (pts (xy 122.174 75.692) (xy 125.73 75.692))
     (stroke (width 0) (type default) (color 0 0 0 0))
   )
-  (label "CELL2" (at 169.418 87.122 0)
+  (wire (pts (xy 94.488 78.994) (xy 99.822 78.994))
+    (stroke (width 0) (type default) (color 0 0 0 0))
+  )
+  (label "4V0" (at 99.822 78.994 180)
+    (effects (font (size 1.27 1.27)) (justify right bottom))
+  )
+  (label "4V1" (at 111.506 78.74 180)
+    (effects (font (size 1.27 1.27)) (justify right bottom))
+  )
+  (label "4V1" (at 119.888 80.772 0)
     (effects (font (size 1.27 1.27)) (justify left bottom))
   )
-  (label "CELL1" (at 169.418 84.582 0)
+  (label "4V0" (at 119.888 78.232 0)
     (effects (font (size 1.27 1.27)) (justify left bottom))
   )
-  (label "CELL3" (at 119.888 83.312 0)
-    (effects (font (size 1.27 1.27)) (justify left bottom))
-  )
-  (label "VT" (at 119.888 85.852 0)
-    (effects (font (size 1.27 1.27)) (justify left bottom))
-  )
-  (label "CELL2" (at 119.888 80.772 0)
-    (effects (font (size 1.27 1.27)) (justify left bottom))
-  )
-  (label "CELL3" (at 169.418 89.662 0)
-    (effects (font (size 1.27 1.27)) (justify left bottom))
-  )
-  (label "CELL1" (at 119.888 78.232 0)
-    (effects (font (size 1.27 1.27)) (justify left bottom))
-  )
-  (label "VT" (at 169.418 92.202 0)
-    (effects (font (size 1.27 1.27)) (justify left bottom))
-  )
   (hierarchical_label "3.3V" (shape input) (at 121.412 101.092 180)
+    (effects (font (size 1.27 1.27)) (justify right))
+  )
+  (hierarchical_label "VCC0" (shape input) (at 94.488 71.374 180)
     (effects (font (size 1.27 1.27)) (justify right))
   )
@@
     (effects (font (size 1.27 1.27)) (justify right))
   )
-  (symbol (lib_id "24V_Li_batt:Conn_01x04") (at 180.34 87.122 0) (unit 1)
-    (in_bom yes) (on_board yes) (fields_autoplaced)
-    (property "Reference" "J9" (id 0) (at 183.134 87.1219 0)
-      (effects (font (size 1.27 1.27)) (justify left))
-    )
-    (property "Value" "JST-BATT" (id 1) (at 183.134 89.6619 0)
-      (effects (font (size 1.27 1.27)) (justify left))
-    )
-    (property "Footprint" "Connector_PinHeader_2.54mm:PinHeader_1x04_P2.54mm_Vertical" (id 2) (at 180.34 87.122 0)
-      (effects (font (size 1.27 1.27)) hide)
-    )
-    (property "Datasheet" "~" (id 3) (at 180.34 87.122 0)
-      (effects (font (size 1.27 1.27)) hide)
-    )
-    (pin "1")
-    (pin "2")
-    (pin "3")
-    (pin "4")
+  (hierarchical_label "VCC1" (shape input) (at 106.172 71.12 180)
+    (effects (font (size 1.27 1.27)) (justify right))
+  )
+  (symbol (lib_id "Device:R_US") (at 94.488 82.804 0) (unit 1)
+    (in_bom yes) (on_board yes) (fields_autoplaced)
+    (property "Reference" "R8" (id 0) (at 96.52 81.5339 0)
+      (effects (font (size 1.27 1.27)) (justify left))
+    )
+    (property "Value" "1k" (id 1) (at 96.52 84.0739 0)
+      (effects (font (size 1.27 1.27)) (justify left))
+    )
+    (property "Footprint" "Resistor_SMD:R_0805_2012Metric_Pad1.20x1.40mm_HandSolder" (id 2) (at 95.504 83.058 90)
+      (effects (font (size 1.27 1.27)) hide)
+    )
+    (property "Datasheet" "https://www.digikey.com/en/products/detail/te-connectivity-passive-product/RA73F2A1K0BTD/16031399" (id 3) (at 94.488 82.804 0)
+      (effects (font (size 1.27 1.27)) hide)
+    )
+    (pin "1")
+    (pin "2")
   )
   (symbol (lib_id "power:GND") (at 161.29 111.252 90) (unit 1)
@@
     )
     (pin "1")
+  )
+  (symbol (lib_id "power:GND") (at 94.488 86.614 0) (unit 1)
+    (in_bom yes) (on_board yes) (fields_autoplaced)
+    (property "Reference" "#PWR0110" (id 0) (at 94.488 92.964 0)
+      (effects (font (size 1.27 1.27)) hide)
+    )
+    (property "Value" "GND" (id 1) (at 94.488 91.694 0))
+    (property "Footprint" "" (id 2) (at 94.488 86.614 0)
+      (effects (font (size 1.27 1.27)) hide)
+    )
+    (property "Datasheet" "" (id 3) (at 94.488 86.614 0)
+      (effects (font (size 1.27 1.27)) hide)
+    )
+    (pin "1")
+  )
+  (symbol (lib_id "Device:R_US") (at 106.172 82.55 0) (unit 1)
+    (in_bom yes) (on_board yes) (fields_autoplaced)
+    (property "Reference" "R6" (id 0) (at 107.95 81.2799 0)
+      (effects (font (size 1.27 1.27)) (justify left))
+    )
+    (property "Value" "1k" (id 1) (at 107.95 83.8199 0)
+      (effects (font (size 1.27 1.27)) (justify left))
+    )
+    (property "Footprint" "Resistor_SMD:R_0805_2012Metric_Pad1.20x1.40mm_HandSolder" (id 2) (at 107.188 82.804 90)
+      (effects (font (size 1.27 1.27)) hide)
+    )
+    (property "Datasheet" "https://www.digikey.com/en/products/detail/te-connectivity-passive-product/RA73F2A1K0BTD/16031399" (id 3) (at 106.172 82.55 0)
+      (effects (font (size 1.27 1.27)) hide)
+    )
+    (pin "1")
+    (pin "2")
   )
   (symbol (lib_id "MCP3008-I_SL:MCP3008-I{slash}SL") (at 143.51 90.932 0) (unit 1)
@@
     (pin "9")
   )
+  (symbol (lib_id "Device:R_US") (at 106.172 74.93 0) (unit 1)
+    (in_bom yes) (on_board yes) (fields_autoplaced)
+    (property "Reference" "R1" (id 0) (at 107.95 73.6599 0)
+      (effects (font (size 1.27 1.27)) (justify left))
+    )
+    (property "Value" "2k" (id 1) (at 107.95 76.1999 0)
+      (effects (font (size 1.27 1.27)) (justify left))
+    )
+    (property "Footprint" "Resistor_SMD:R_0805_2012Metric_Pad1.20x1.40mm_HandSolder" (id 2) (at 107.188 75.184 90)
+      (effects (font (size 1.27 1.27)) hide)
+    )
+    (property "Datasheet" "https://www.digikey.com/en/products/detail/te-connectivity-passive-product/RA73F2A2K0BTD/16031942" (id 3) (at 106.172 74.93 0)
+      (effects (font (size 1.27 1.27)) hide)
+    )
+    (pin "1")
+    (pin "2")
+  )
   (symbol (lib_id "power:GND") (at 161.29 108.712 90) (unit 1)
     (in_bom yes) (on_board yes) (fields_autoplaced)
@@
     (pin "1")
   )
+  (symbol (lib_id "Device:R_US") (at 94.488 75.184 0) (unit 1)
+    (in_bom yes) (on_board yes) (fields_autoplaced)
+    (property "Reference" "R7" (id 0) (at 96.52 73.9139 0)
+      (effects (font (size 1.27 1.27)) (justify left))
+    )
+    (property "Value" "2k" (id 1) (at 96.52 76.4539 0)
+      (effects (font (size 1.27 1.27)) (justify left))
+    )
+    (property "Footprint" "Resistor_SMD:R_0805_2012Metric_Pad1.20x1.40mm_HandSolder" (id 2) (at 95.504 75.438 90)
+      (effects (font (size 1.27 1.27)) hide)
+    )
+    (property "Datasheet" "https://www.digikey.com/en/products/detail/te-connectivity-passive-product/RA73F2A2K0BTD/16031942" (id 3) (at 94.488 75.184 0)
+      (effects (font (size 1.27 1.27)) hide)
+    )
+    (pin "1")
+    (pin "2")
+  )
   (symbol (lib_id "power:PWR_FLAG") (at 161.29 68.072 0) (unit 1)
     (in_bom yes) (on_board yes) (fields_autoplaced)
@@
       (effects (font (size 1.27 1.27)) hide)
     )
+    (pin "1")
+  )
+  (symbol (lib_id "power:GND") (at 106.172 86.36 0) (unit 1)
+    (in_bom yes) (on_board yes) (fields_autoplaced)
+    (property "Reference" "#PWR0105" (id 0) (at 106.172 92.71 0)
+      (effects (font (size 1.27 1.27)) hide)
+    )
+    (property "Value" "GND" (id 1) (at 106.172 91.44 0))
+    (property "Footprint" "" (id 2) (at 106.172 86.36 0)
+      (effects (font (size 1.27 1.27)) hide)
+    )
+    (property "Datasheet" "" (id 3) (at 106.172 86.36 0)
+      (effects (font (size 1.27 1.27)) hide)
+    )
