File: ISAAC/PCB/Pi_HAT/V3/Pi_HAT_V3/Buck Converter.kicad_sch (KiCad schematic)
At the start: 21 parts, among them J4 Conn_01x04_Male, J5 XT60PW-M, J6 Conn_01x04_Male, J8 XT60PW-M, U1 MP2315GJ-Z

Commit message: Final Updates "HOPEFULLY"
Connections:
- net +12V renamed VCC1
- net VCC1: no longer J4.1 (Pin_1), J5.1 (+), J6.1 (Pin_1)
- new net VCC0: J4.1 (Pin_1), J5.1 (+), J6.1 (Pin_1)
Changed lines of the file:
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@@
   (junction (at 110.49 41.91) (diameter 0) (color 0 0 0 0)
   )
-  (junction (at 83.82 81.28) (diameter 0) (color 0 0 0 0)
-  )
   (junction (at 194.31 67.31) (diameter 0) (color 0 0 0 0)
   )
   (junction (at 87.63 81.28) (diameter 0) (color 0 0 0 0)
   )
+  (junction (at 114.3 44.45) (diameter 0) (color 0 0 0 0)
+  )
   (junction (at 173.99 92.71) (diameter 0) (color 0 0 0 0)
   )
@@
   (junction (at 215.9 67.31) (diameter 0) (color 0 0 0 0)
   )
-  (junction (at 116.84 45.72) (diameter 0) (color 0 0 0 0)
-  )
   (junction (at 96.52 81.28) (diameter 0) (color 0 0 0 0)
   )
@@
     (stroke (width 0) (type default) (color 0 0 0 0))
   )
+  (wire (pts (xy 114.3 41.91) (xy 114.3 44.45))
+    (stroke (width 0) (type default) (color 0 0 0 0))
+  )
   (wire (pts (xy 154.94 67.31) (xy 158.75 67.31))
     (stroke (width 0) (type default) (color 0 0 0 0))
@@
     (stroke (width 0) (type default) (color 0 0 0 0))
   )
+  (wire (pts (xy 114.3 44.45) (xy 116.84 44.45))
+    (stroke (width 0) (type default) (color 0 0 0 0))
+  )
   (wire (pts (xy 166.37 67.31) (xy 170.18 67.31))
     (stroke (width 0) (type default) (color 0 0 0 0))
   )
-  (wire (pts (xy 114.3 41.91) (xy 114.3 45.72))
-    (stroke (width 0) (type default) (color 0 0 0 0))
-  )
   (wire (pts (xy 143.51 81.28) (xy 166.37 81.28))
     (stroke (width 0) (type default) (color 0 0 0 0))
@@
     (stroke (width 0) (type default) (color 0 0 0 0))
   )
-  (wire (pts (xy 83.82 35.56) (xy 83.82 81.28))
-    (stroke (width 0) (type default) (color 0 0 0 0))
-  )
-  (wire (pts (xy 116.84 44.45) (xy 116.84 45.72))
+  (wire (pts (xy 83.82 35.56) (xy 83.82 41.148))
     (stroke (width 0) (type default) (color 0 0 0 0))
   )
@@
     (stroke (width 0) (type default) (color 0 0 0 0))
   )
-  (wire (pts (xy 114.3 45.72) (xy 116.84 45.72))
-    (stroke (width 0) (type default) (color 0 0 0 0))
-  )
   (wire (pts (xy 87.63 81.28) (xy 96.52 81.28))
     (stroke (width 0) (type default) (color 0 0 0 0))
   )
+  (wire (pts (xy 132.588 44.45) (xy 132.588 47.498))
+    (stroke (width 0) (type default) (color 0 0 0 0))
+  )
   (wire (pts (xy 182.88 67.31) (xy 194.31 67.31))
     (stroke (width 0) (type default) (color 0 0 0 0))
@@
   )
   (wire (pts (xy 153.67 92.71) (xy 166.37 92.71))
+    (stroke (width 0) (type default) (color 0 0 0 0))
+  )
+  (wire (pts (xy 75.438 41.148) (xy 83.82 41.148))
     (stroke (width 0) (type default) (color 0 0 0 0))
   )
@@
     (effects (font (size 2 2)) (justify left bottom))
   )
-  (global_label "12V" (shape input) (at 114.3 45.72 180) (fields_autoplaced)
+  (label "12V" (at 132.588 47.498 180)
+    (effects (font (size 1.27 1.27)) (justify right bottom))
+  )
+  (label "12V" (at 83.82 81.28 180)
+    (effects (font (size 1.27 1.27)) (justify right bottom))
+  )
+  (hierarchical_label "VCC0" (shape input) (at 116.84 44.45 270)
     (effects (font (size 1.27 1.27)) (justify right))
-    (property "Intersheet References" "${INTERSHEET_REFS}" (id 0) (at -9.652 -0.762 0)
-      (effects (font (size 1.27 1.27)) hide)
-    )
-  )
-  (global_label "12V" (shape input) (at 75.438 41.148 0) (fields_autoplaced)
-    (effects (font (size 1.27 1.27)) (justify left))
-    (property "Intersheet References" "${INTERSHEET_REFS}" (id 0) (at 199.39 87.63 0)
-      (effects (font (size 1.27 1.27)) hide)
-    )
-  )
-  (global_label "12V" (shape input) (at 132.588 44.45 180) (fields_autoplaced)
-    (effects (font (size 1.27 1.27)) (justify right))
-    (property "Intersheet References" "${INTERSHEET_REFS}" (id 0) (at 8.636 -2.032 0)
-      (effects (font (size 1.27 1.27)) hide)
-    )
   )
   (hierarchical_label "SCL" (shape input) (at 75.438 46.228 0)
@@
     (effects (font (size 1.27 1.27)) (justify left))
   )
+  (hierarchical_label "VCC1" (shape input) (at 132.588 44.45 180)
+    (effects (font (size 1.27 1.27)) (justify right))
+  )
   (symbol (lib_id "power:GND") (at 119.38 44.45 0) (unit 1)
     (in_bom yes) (on_board yes)
@@
     (pin "1")
     (pin "2")
-  )
-  (symbol (lib_id "power:+12V") (at 132.588 44.45 180) (unit 1)
-    (in_bom yes) (on_board yes)
-    (property "Reference" "#PWR0110" (id 0) (at 132.588 40.64 0)
-      (effects (font (size 1.27 1.27)) hide)
-    )
-    (property "Value" "~" (id 1) (at 132.588 48.895 0))
-    (property "Footprint" "" (id 2) (at 132.588 44.45 0)
-      (effects (font (size 1.27 1.27)) hide)
-    )
-    (property "Datasheet" "" (id 3) (at 132.588 44.45 0)
-      (effects (font (size 1.27 1.27)) hide)
-    )
-    (pin "1")
   )
   (symbol (lib_id "Device:R_US") (at 170.18 92.71 270) (unit 1)
@@
     (pin "4")
   )
+  (symbol (lib_id "power:PWR_FLAG") (at 114.3 44.45 0) (unit 1)
+    (in_bom yes) (on_board yes)
+    (property "Reference" "#FLG0101" (id 0) (at 114.3 42.545 0)
+      (effects (font (size 1.27 1.27)) hide)
+    )
+    (property "Value" "PWR_FLAG" (id 1) (at 114.3 40.894 0))
+    (property "Footprint" "" (id 2) (at 114.3 44.45 0)
+      (effects (font (size 1.27 1.27)) hide)
+    )
+    (property "Datasheet" "~" (id 3) (at 114.3 44.45 0)
+      (effects (font (size 1.27 1.27)) hide)
+    )
+    (pin "1")
+  )
   (symbol (lib_id "Device:R_US") (at 100.33 91.44 90) (unit 1)
     (in_bom yes) (on_board yes)
@@
     (pin "1")
     (pin "2")
-  )
-  (symbol (lib_id "power:PWR_FLAG") (at 116.84 45.72 180) (unit 1)
-    (in_bom yes) (on_board yes)
-    (property "Reference" "#FLG0101" (id 0) (at 116.84 47.625 0)
-      (effects (font (size 1.27 1.27)) hide)
-    )
-    (property "Value" "PWR_FLAG" (id 1) (at 116.84 50.1142 0))
-    (property "Footprint" "" (id 2) (at 116.84 45.72 0)
-      (effects (font (size 1.27 1.27)) hide)
-    )
-    (property "Datasheet" "~" (id 3) (at 116.84 45.72 0)
-      (effects (font (size 1.27 1.27)) hide)
-    )
-    (pin "1")
   )
   (symbol (lib_id "power:GND") (at 107.95 58.42 180) (unit 1)
@@
     (pin "2")
   )
-  (symbol (lib_id "power:+12V") (at 116.84 45.72 180) (unit 1)
-    (in_bom yes) (on_board yes)
-    (property "Reference" "#PWR0105" (id 0) (at 116.84 41.91 0)
-      (effects (font (size 1.27 1.27)) hide)
-    )
-    (property "Value" "~" (id 1) (at 116.84 50.165 0))
-    (property "Footprint" "" (id 2) (at 116.84 45.72 0)
-      (effects (font (size 1.27 1.27)) hide)
-    )
-    (property "Datasheet" "" (id 3) (at 116.84 45.72 0)
-      (effects (font (size 1.27 1.27)) hide)
-    )
-    (pin "1")
-  )
   (symbol (lib_id "Connector:Conn_01x04_Male") (at 93.98 44.45 0) (unit 1)
