File: ISAAC/PCB/Pi_HAT/V3/Pi_HAT_V3/Pi_HAT_V3.kicad_pcb (KiCad board)
At the start: 2 copper layers, 71.7 x 71.3 mm, 30 parts, among them J1 MPU 6050, J2 Pi_GPIO, J3 Display, J4 Conn_01x04_Male, J5 XT60PW-M, J6 Conn_01x04_Male, J7 Pressure Sensor, J8 XT60PW-M, U1 MP2315GJ-Z, U2 MCP3008-I/SL

Commit message: Traced V3
Routing:
- net 12V: track 0.00 -> 184.8 mm, vias 0 -> 1
- net /SCL: track 0.00 -> 131.6 mm
- net /SDA: track 0.00 -> 130.8 mm
- net /5V: track 0.00 -> 118.5 mm
- net GND: track 0.00 -> 91.8 mm, vias 0 -> 4
- net Net-(C5-Pad1): track 0.00 -> 68.0 mm, vias 0 -> 3
- net /3.3V: track 0.00 -> 63.1 mm, vias 0 -> 1
- net /PS: track 0.00 -> 41.7 mm, vias 0 -> 2
- net /SCLK: track 0.00 -> 24.0 mm, vias 0 -> 1
- net /MISO: track 0.00 -> 19.7 mm, vias 0 -> 1
- net /CS: track 0.00 -> 18.1 mm, vias 0 -> 2
- net /MOSI: track 0.00 -> 18.0 mm, vias 0 -> 1
- net Net-(C4-Pad1): track 0.00 -> 17.8 mm, vias 0 -> 2
- net Net-(R3-Pad1): track 0.00 -> 13.7 mm, vias 0 -> 2
- net Net-(R4-Pad1): track 0.00 -> 9.76 mm
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- added copper zone on B.Cu, net GND
- removed copper zone on F.Cu, net GND

Commit message: Uploaded Gerber
Routing:
- net Net-(C5-Pad1): track 68.0 -> 68.9 mm

Commit message: Shit ton of stuf
Parts:
- removed J8: XT60PW-M, .pretty:AMASS_XT60PW-M
- added G***: LOGO, .pretty:eppl_logo, F.Cu at (136.9, 85.1)
- added J9: JST-BATT, Connector_PinHeader_2.54mm:PinHeader_1x04_P2.54mm_Vertical, F.Cu at (104.9, 68.2)
- moved J1 7.05 mm to (129.9, 114.0)
Connections:
- J2 pad 10: /RXP -> unconnected-(J2-Pad10)
- J2 pad 22: /CS -> unconnected-(J2-Pad22)
- J2 pad 24: /SCLK -> /CS
- J2 pad 8: /TXP -> unconnected-(J2-Pad8)
- U2 pad 2: unconnected-(U2-Pad2) -> /A-D Converter/CELL1
- U2 pad 3: unconnected-(U2-Pad3) -> /A-D Converter/CELL2
- U2 pad 4: unconnected-(U2-Pad4) -> /A-D Converter/CELL3
- U2 pad 5: unconnected-(U2-Pad5) -> /A-D Converter/VT
Routing:
- net /A-D Converter/VT: track 0.00 -> 59.8 mm
- net /A-D Converter/CELL3: track 0.00 -> 57.8 mm
- net /A-D Converter/CELL2: track 0.00 -> 56.8 mm
- net /A-D Converter/CELL1: track 0.00 -> 56.4 mm
- net GND: track 91.8 -> 144.4 mm, vias 4 -> 3
- net 12V: track 184.8 -> 162.6 mm, vias 1 -> 0
- net /3.3V: track 63.1 -> 78.0 mm
- net /SCL: track 131.9 -> 141.3 mm
- net /SDA: track 130.8 -> 140.0 mm
- net /5V: track 118.5 -> 125.1 mm
- net Net-(C5-Pad1): track 68.9 -> 73.5 mm, vias 3 -> 2
- net /PS: track 41.7 -> 37.5 mm, vias 2 -> 1
- net /CS: track 18.1 -> 21.6 mm, vias 2 -> 1
- net /SCLK: track 24.0 -> 21.4 mm

Commit message: Final Updates "HOPEFULLY"
Parts:
- removed J9: JST-BATT, Connector_PinHeader_2.54mm:PinHeader_1x04_P2.54mm_Vertical
- added J8: XT60PW-M, .pretty:AMASS_XT60PW-M, F.Cu at (117.4, 125.1)
- added R1: 2k, Resistor_SMD:R_0805_2012Metric_Pad1.20x1.40mm_HandSolder, B.Cu at (128.4, 96.7)
- added R6: 1k, Resistor_SMD:R_0805_2012Metric_Pad1.20x1.40mm_HandSolder, B.Cu at (130.7, 96.7)
- added R7: 2k, Resistor_SMD:R_0805_2012Metric_Pad1.20x1.40mm_HandSolder, B.Cu at (126.6, 92.2)
- added R8: 1k, Resistor_SMD:R_0805_2012Metric_Pad1.20x1.40mm_HandSolder, B.Cu at (129.0, 92.2)
- moved G*** 7.51 mm to (138.1, 92.5), turned to -45 degrees
Connections:
- C1 pad 1: 12V -> /12V1
- C2 pad 1: 12V -> /12V1
- J4 pad 1: 12V -> /12V0
- J5 pad 1: 12V -> /12V0
- J6 pad 1: 12V -> /12V0
- R2 pad 1: 12V -> /12V1
- U1 pad 2: 12V -> /12V1
- U2 pad 2: /A-D Converter/CELL1 -> /A-D Converter/4V0
- U2 pad 3: /A-D Converter/CELL2 -> /A-D Converter/4V1
- U2 pad 4: /A-D Converter/CELL3 -> unconnected-(U2-Pad4)
- U2 pad 5: /A-D Converter/VT -> unconnected-(U2-Pad5)
Routing:
- net 12V: track 162.6 -> 0.00 mm
- net /12V0: track 0.00 -> 138.0 mm
- net /12V1: track 0.00 -> 68.0 mm, vias 0 -> 2
- net /A-D Converter/VT: track 59.8 -> 0.00 mm
- net /A-D Converter/CELL3: track 57.8 -> 0.00 mm
- net /A-D Converter/CELL2: track 56.8 -> 0.00 mm
- net /A-D Converter/CELL1: track 56.4 -> 0.00 mm
- net /A-D Converter/4V1: track 0.00 -> 10.1 mm
- net /A-D Converter/4V0: track 0.00 -> 9.49 mm
- net Net-(C5-Pad1): track 73.5 -> 66.6 mm
- net GND: track 144.4 -> 150.5 mm
- net /3.3V: track 78.0 -> 80.1 mm
- net /5V: track 125.1 -> 125.7 mm
Other:
- board text added: "PS"
