File: ISAAC/PCB/Pi_HAT/V3/Pi_HAT_V3_simple/A-D Converter.kicad_sch (KiCad schematic)
At the start: 3 parts, among them J5 Pressure Sensor, J6 JST-BATT, U2 MCP3008-I/SL

Commit message: Final Updates "HOPEFULLY"
Parts:
- removed J6: JST-BATT, Connector_PinHeader_2.54mm:PinHeader_1x04_P2.54mm_Vertical, symbol 24V_Li_batt:Conn_01x04
- added R1: 2k, Resistor_SMD:R_0805_2012Metric_Pad1.20x1.40mm_HandSolder, symbol Device:R_US
- added R2: 1k, Resistor_SMD:R_0805_2012Metric_Pad1.20x1.40mm_HandSolder, symbol Device:R_US
Connections:
- net GND: now also R2.2
- net CELL1 renamed 4V
- net 4V: now also R1.2, R2.1
- net CELL2: no longer names the net of U2.3 (CH2)
- net CELL3: no longer names the net of U2.4 (CH3)
- net VT: no longer names the net of U2.5 (CH4)
- new net VCC: R1.1
- no-connect marks 3 -> 6
Other:
- moved on the sheet: J5
Changed lines of the file:
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@@
   (junction (at 161.29 68.072) (diameter 0) (color 0 0 0 0)
+  )
+  (junction (at 103.632 80.518) (diameter 0) (color 0 0 0 0)
   )
   (no_connect (at 125.73 88.392))
   (no_connect (at 125.73 90.932))
   (no_connect (at 125.73 93.472))
-  (wire (pts (xy 120.142 83.312) (xy 125.73 83.312))
-    (stroke (width 0) (type default) (color 0 0 0 0))
-  )
+  (no_connect (at 125.73 83.312))
+  (no_connect (at 125.73 85.852))
+  (no_connect (at 125.73 80.772))
   (wire (pts (xy 161.29 73.152) (xy 165.608 73.152))
     (stroke (width 0) (type default) (color 0 0 0 0))
@@
     (stroke (width 0) (type default) (color 0 0 0 0))
   )
-  (wire (pts (xy 171.704 89.408) (xy 177.546 89.408))
-    (stroke (width 0) (type default) (color 0 0 0 0))
-  )
   (wire (pts (xy 125.73 101.092) (xy 121.412 101.092))
     (stroke (width 0) (type default) (color 0 0 0 0))
   )
-  (wire (pts (xy 171.704 91.948) (xy 177.546 91.948))
-    (stroke (width 0) (type default) (color 0 0 0 0))
-  )
-  (wire (pts (xy 171.704 86.868) (xy 177.546 86.868))
-    (stroke (width 0) (type default) (color 0 0 0 0))
-  )
   (wire (pts (xy 122.174 73.152) (xy 125.73 73.152))
     (stroke (width 0) (type default) (color 0 0 0 0))
   )
+  (wire (pts (xy 103.632 80.518) (xy 108.966 80.518))
+    (stroke (width 0) (type default) (color 0 0 0 0))
+  )
   (wire (pts (xy 120.142 78.232) (xy 125.73 78.232))
     (stroke (width 0) (type default) (color 0 0 0 0))
   )
-  (wire (pts (xy 177.546 81.28) (xy 172.466 81.28))
-    (stroke (width 0) (type default) (color 0 0 0 0))
-  )
-  (wire (pts (xy 120.142 80.772) (xy 125.73 80.772))
-    (stroke (width 0) (type default) (color 0 0 0 0))
-  )
-  (wire (pts (xy 120.142 85.852) (xy 125.73 85.852))
-    (stroke (width 0) (type default) (color 0 0 0 0))
-  )
-  (wire (pts (xy 177.546 76.2) (xy 172.466 76.2))
+  (wire (pts (xy 173.482 92.964) (xy 168.402 92.964))
+    (stroke (width 0) (type default) (color 0 0 0 0))
+  )
+  (wire (pts (xy 173.482 87.884) (xy 168.402 87.884))
     (stroke (width 0) (type default) (color 0 0 0 0))
   )
@@
     (stroke (width 0) (type default) (color 0 0 0 0))
   )
-  (wire (pts (xy 171.704 94.488) (xy 177.546 94.488))
-    (stroke (width 0) (type default) (color 0 0 0 0))
-  )
   (wire (pts (xy 161.29 68.072) (xy 165.608 68.072))
     (stroke (width 0) (type default) (color 0 0 0 0))
   )
-  (label "CELL3" (at 171.704 91.948 0)
+  (label "PS" (at 168.402 92.964 0)
     (effects (font (size 1.27 1.27)) (justify left bottom))
   )
-  (label "VT" (at 120.142 85.852 0)
-    (effects (font (size 1.27 1.27)) (justify left bottom))
-  )
-  (label "CELL1" (at 171.704 86.868 0)
-    (effects (font (size 1.27 1.27)) (justify left bottom))
-  )
-  (label "PS" (at 172.466 81.28 0)
-    (effects (font (size 1.27 1.27)) (justify left bottom))
-  )
-  (label "CELL1" (at 120.142 78.232 0)
-    (effects (font (size 1.27 1.27)) (justify left bottom))
-  )
-  (label "VT" (at 171.704 94.488 0)
-    (effects (font (size 1.27 1.27)) (justify left bottom))
-  )
-  (label "CELL3" (at 120.142 83.312 0)
-    (effects (font (size 1.27 1.27)) (justify left bottom))
-  )
-  (label "CELL2" (at 120.142 80.772 0)
+  (label "4V" (at 108.966 80.518 180)
+    (effects (font (size 1.27 1.27)) (justify right bottom))
+  )
+  (label "4V" (at 120.142 78.232 0)
     (effects (font (size 1.27 1.27)) (justify left bottom))
   )
@@
     (effects (font (size 1.27 1.27)) (justify left bottom))
   )
-  (label "CELL2" (at 171.704 89.408 0)
-    (effects (font (size 1.27 1.27)) (justify left bottom))
-  )
   (hierarchical_label "3.3V" (shape input) (at 121.412 101.092 180)
     (effects (font (size 1.27 1.27)) (justify right))
@@
     (effects (font (size 1.27 1.27)) (justify left))
   )
+  (hierarchical_label "VCC" (shape input) (at 103.632 72.898 180)
+    (effects (font (size 1.27 1.27)) (justify right))
+  )
   (hierarchical_label "SCLK" (shape input) (at 121.412 96.012 180)
     (effects (font (size 1.27 1.27)) (justify right))
@@
     (effects (font (size 1.27 1.27)) (justify left))
   )
-  (hierarchical_label "5V" (shape input) (at 172.466 76.2 180)
+  (hierarchical_label "5V" (shape input) (at 168.402 87.884 180)
     (effects (font (size 1.27 1.27)) (justify right))
   )
@@
     (pin "9")
   )
-  (symbol (lib_id "24V_Li_batt:Conn_01x04") (at 182.626 89.408 0) (unit 1)
-    (in_bom yes) (on_board yes) (fields_autoplaced)
-    (property "Reference" "J6" (id 0) (at 185.42 89.4079 0)
-      (effects (font (size 1.27 1.27)) (justify left))
-    )
-    (property "Value" "JST-BATT" (id 1) (at 185.42 91.9479 0)
-      (effects (font (size 1.27 1.27)) (justify left))
-    )
-    (property "Footprint" "Connector_PinHeader_2.54mm:PinHeader_1x04_P2.54mm_Vertical" (id 2) (at 182.626 89.408 0)
-      (effects (font (size 1.27 1.27)) hide)
-    )
-    (property "Datasheet" "~" (id 3) (at 182.626 89.408 0)
-      (effects (font (size 1.27 1.27)) hide)
-    )
-    (pin "1")
-    (pin "2")
-    (pin "3")
-    (pin "4")
-  )
-  (symbol (lib_id "power:GND") (at 177.546 78.74 270) (unit 1)
+  (symbol (lib_id "power:GND") (at 173.482 90.424 270) (unit 1)
     (in_bom yes) (on_board yes)
-    (property "Reference" "#PWR0104" (id 0) (at 171.196 78.74 0)
-      (effects (font (size 1.27 1.27)) hide)
-    )
-    (property "Value" "GND" (id 1) (at 175.006 78.232 90)
+    (property "Reference" "#PWR0104" (id 0) (at 167.132 90.424 0)
+      (effects (font (size 1.27 1.27)) hide)
+    )
+    (property "Value" "GND" (id 1) (at 170.942 89.916 90)
       (effects (font (size 1.27 1.27)) (justify right))
     )
-    (property "Footprint" "" (id 2) (at 177.546 78.74 0)
-      (effects (font (size 1.27 1.27)) hide)
-    )
-    (property "Datasheet" "" (id 3) (at 177.546 78.74 0)
+    (property "Footprint" "" (id 2) (at 173.482 90.424 0)
+      (effects (font (size 1.27 1.27)) hide)
+    )
+    (property "Datasheet" "" (id 3) (at 173.482 90.424 0)
+      (effects (font (size 1.27 1.27)) hide)
+    )
+    (pin "1")
+  )
+  (symbol (lib_id "power:GND") (at 103.632 88.138 0) (unit 1)
+    (in_bom yes) (on_board yes) (fields_autoplaced)
+    (property "Reference" "#PWR0105" (id 0) (at 103.632 94.488 0)
+      (effects (font (size 1.27 1.27)) hide)
+    )
+    (property "Value" "GND" (id 1) (at 103.632 93.218 0))
+    (property "Footprint" "" (id 2) (at 103.632 88.138 0)
+      (effects (font (size 1.27 1.27)) hide)
+    )
+    (property "Datasheet" "" (id 3) (at 103.632 88.138 0)
       (effects (font (size 1.27 1.27)) hide)
     )
@@
     (pin "1")
   )
-  (symbol (lib_id "Connector_Generic:Conn_01x03") (at 182.626 78.74 0) (unit 1)
+  (symbol (lib_id "Device:R_US") (at 103.632 76.708 0) (unit 1)
+    (in_bom yes) (on_board yes) (fields_autoplaced)
+    (property "Reference" "R1" (id 0) (at 105.41 75.4379 0)
+      (effects (font (size 1.27 1.27)) (justify left))
+    )
+    (property "Value" "2k" (id 1) (at 105.41 77.9779 0)
+      (effects (font (size 1.27 1.27)) (justify left))
+    )
+    (property "Footprint" "Resistor_SMD:R_0805_2012Metric_Pad1.20x1.40mm_HandSolder" (id 2) (at 104.648 76.962 90)
+      (effects (font (size 1.27 1.27)) hide)
+    )
+    (property "Datasheet" "https://www.digikey.com/en/products/detail/te-connectivity-passive-product/RA73F2A2K0BTD/16031942" (id 3) (at 103.632 76.708 0)
+      (effects (font (size 1.27 1.27)) hide)
+    )
+    (pin "1")
+    (pin "2")
+  )
+  (symbol (lib_id "Connector_Generic:Conn_01x03") (at 178.562 90.424 0) (unit 1)
     (in_bom yes) (on_board yes)
-    (property "Reference" "J5" (id 0) (at 182.372 71.12 0))
-    (property "Value" "Pressure Sensor" (id 1) (at 182.372 72.898 0))
-    (property "Footprint" "Connector_PinHeader_2.54mm:PinHeader_1x03_P2.54mm_Vertical" (id 2) (at 182.626 78.74 0)
-      (effects (font (size 1.27 1.27)) hide)
-    )
-    (property "Datasheet" "https://www.te.com/commerce/DocumentDelivery/DDEController?Action=srchrtrv&DocNm=MSP340&DocType=Data+Sheet&DocLang=English" (id 3) (at 182.626 78.74 0)
+    (property "Reference" "J5" (id 0) (at 178.308 82.804 0))
+    (property "Value" "Pressure Sensor" (id 1) (at 178.308 84.582 0))
+    (property "Footprint" "Connector_PinHeader_2.54mm:PinHeader_1x03_P2.54mm_Vertical" (id 2) (at 178.562 90.424 0)
+      (effects (font (size 1.27 1.27)) hide)
+    )
+    (property "Datasheet" "https://www.te.com/commerce/DocumentDelivery/DDEController?Action=srchrtrv&DocNm=MSP340&DocType=Data+Sheet&DocLang=English" (id 3) (at 178.562 90.424 0)
       (effects (font (size 1.27 1.27)) hide)
     )
@@
     (pin "3")
   )
+  (symbol (lib_id "Device:R_US") (at 103.632 84.328 0) (unit 1)
+    (in_bom yes) (on_board yes) (fields_autoplaced)
+    (property "Reference" "R2" (id 0) (at 105.41 83.0579 0)
+      (effects (font (size 1.27 1.27)) (justify left))
+    )
+    (property "Value" "1k" (id 1) (at 105.41 85.5979 0)
+      (effects (font (size 1.27 1.27)) (justify left))
+    )
+    (property "Footprint" "Resistor_SMD:R_0805_2012Metric_Pad1.20x1.40mm_HandSolder" (id 2) (at 104.648 84.582 90)
+      (effects (font (size 1.27 1.27)) hide)
+    )
+    (property "Datasheet" "https://www.digikey.com/en/products/detail/te-connectivity-passive-product/RA73F2A1K0BTD/16031399" (id 3) (at 103.632 84.328 0)
+      (effects (font (size 1.27 1.27)) hide)
+    )
+    (pin "1")
+    (pin "2")
+  )
   (symbol (lib_id "power:PWR_FLAG") (at 161.29 68.072 0) (unit 1)
