File: ISAAC/PCB/Pi_HAT/V3/Pi_HAT_V3_simple/Pi_HAT_Simple_V3.kicad_pcb (KiCad board)
At the start: 2 copper layers, 68.7 x 71.3 mm, 15 parts, among them J1 MPU 6050, J2 Pi_GPIO, J3 Display, J4 INPUT-XT60, J5 Pressure Sensor, J6 JST-BATT, J8 Conn_01x04_Male, J9 Conn_01x04_Male, U1 LM2596S, U2 MCP3008-I/SL

Commit message: Final Updates "HOPEFULLY"
Parts:
- removed J6: JST-BATT, Connector_PinHeader_2.54mm:PinHeader_1x04_P2.54mm_Vertical
- added R1: 2k, Resistor_SMD:R_0805_2012Metric_Pad1.20x1.40mm_HandSolder, B.Cu at (132.2, 101.3)
- added R2: 1k, Resistor_SMD:R_0805_2012Metric_Pad1.20x1.40mm_HandSolder, B.Cu at (135.1, 101.3)
- moved G*** 1.61 mm to (107.7, 91.6)
- moved J5 1.60 mm to (96.7, 73.5)
Connections:
- J4 pad 1: /VCC -> /12V
- J8 pad 1: /VCC -> /12V
- J9 pad 1: /VCC -> /12V
- U2 pad 2: /A-D Converter/CELL1 -> /A-D Converter/4V
- U2 pad 3: /A-D Converter/CELL2 -> unconnected-(U2-Pad3)
- U2 pad 4: /A-D Converter/CELL3 -> unconnected-(U2-Pad4)
- U2 pad 5: /A-D Converter/VT -> unconnected-(U2-Pad5)
Routing:
- net /12V: track 0.00 -> 204.5 mm
- net /VCC: track 177.5 -> 0.00 mm
- net /A-D Converter/CELL1: track 65.9 -> 0.00 mm
- net /A-D Converter/CELL2: track 64.0 -> 0.00 mm
- net /A-D Converter/CELL3: track 63.2 -> 0.00 mm
- net /A-D Converter/VT: track 62.6 -> 0.00 mm
- net GND: track 53.6 -> 36.4 mm
- net /5V: track 91.1 -> 83.3 mm
- net /A-D Converter/4V: track 0.00 -> 7.63 mm
- net /A-D Converter/PS: track 56.0 -> 53.5 mm
Other:
- board text added: "PS"
