File: ISAAC/PCB/Pi_HAT/V3/Pi_HAT_V3_simple/Pi_HAT_Simple_V3.kicad_sch (KiCad schematic)
At the start: 11 parts, among them J1 MPU 6050, J2 Pi_GPIO, J3 Display, J4 INPUT-XT60, J8 Conn_01x04_Male, J9 Conn_01x04_Male, U1 LM2596S

Commit message: Final Updates "HOPEFULLY"
Connections:
- net VCC: no longer J4.1 (+), J8.1 (Pin_1), J9.1 (Pin_1)
- new net 12V: J4.1 (+), J8.1 (Pin_1), J9.1 (Pin_1)
Other:
- sheet A-D Converter ports: added VCC; removed none
Changed lines of the file:
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@@
+    (stroke (width 0) (type default) (color 0 0 0 0))
+  )
+  (wire (pts (xy 179.832 85.852) (xy 184.404 85.852))
     (stroke (width 0) (type default) (color 0 0 0 0))
   )
@@
     (effects (font (size 1.27 1.27)) (justify left bottom))
   )
-  (label "VCC" (at 88.392 88.392 180)
-    (effects (font (size 1.27 1.27)) (justify right bottom))
+  (label "12V" (at 88.392 88.392 180)
+    (effects (font (size 1.27 1.27)) (justify right bottom))
+  )
+  (label "12V" (at 179.832 85.852 0)
+    (effects (font (size 1.27 1.27)) (justify left bottom))
   )
   (label "5V" (at 157.988 59.69 180)
@@
     (effects (font (size 1.27 1.27)) (justify right bottom))
   )
-  (label "VCC" (at 101.092 88.392 180)
+  (label "12V" (at 101.092 88.392 180)
     (effects (font (size 1.27 1.27)) (justify right bottom))
   )
@@
     (effects (font (size 1.27 1.27)) (justify right bottom))
   )
-  (label "VCC" (at 90.424 80.264 90)
+  (label "12V" (at 90.424 80.264 90)
     (effects (font (size 1.27 1.27)) (justify left bottom))
   )
@@
       (effects (font (size 1.27 1.27)) (justify left))
     )
+    (pin "VCC" input (at 184.404 85.852 180)
+      (effects (font (size 1.27 1.27)) (justify left))
+    )
   )
   (sheet_instances
@@
       (reference "#PWR0104") (unit 1) (value "GND") (footprint "")
     )
+    (path "/048aae1f-d538-461c-a17b-6a2498319945/8372ef75-8cab-4e69-bc6b-0af3397ac964"
+      (reference "#PWR0105") (unit 1) (value "GND") (footprint "")
+    )
     (path "/78b7ad88-0121-48a0-a3d1-39a1191d4e39"
       (reference "#PWR0106") (unit 1) (value "GND") (footprint "")
@@
       (reference "J5") (unit 1) (value "Pressure Sensor") (footprint "Connector_PinHeader_2.54mm:PinHeader_1x03_P2.54mm_Vertical")
     )
-    (path "/048aae1f-d538-461c-a17b-6a2498319945/6be0cde9-85b3-4e00-a89d-9afcfe3294f3"
-      (reference "J6") (unit 1) (value "JST-BATT") (footprint "Connector_PinHeader_2.54mm:PinHeader_1x04_P2.54mm_Vertical")
-    )
     (path "/6227afdc-ecf0-4336-bca6-d39069621410"
       (reference "J8") (unit 1) (value "Conn_01x04_Male") (footprint "Connector_PinHeader_2.54mm:PinHeader_1x04_P2.54mm_Vertical")
@@
       (reference "J9") (unit 1) (value "Conn_01x04_Male") (footprint "Connector_PinHeader_2.54mm:PinHeader_1x04_P2.54mm_Vertical")
     )
+    (path "/048aae1f-d538-461c-a17b-6a2498319945/bfebbadf-0ded-4086-99e6-0fdf1796a2da"
+      (reference "R1") (unit 1) (value "2k") (footprint "Resistor_SMD:R_0805_2012Metric_Pad1.20x1.40mm_HandSolder")
+    )
+    (path "/048aae1f-d538-461c-a17b-6a2498319945/d2b89ea4-4495-4fd6-a3ad-6fe88a72acd3"
+      (reference "R2") (unit 1) (value "1k") (footprint "Resistor_SMD:R_0805_2012Metric_Pad1.20x1.40mm_HandSolder")
+    )
     (path "/13fbe27d-eb6a-43f7-a618-c39451faf4f6"
