File: ISAAC/PCB/Pi_HAT/V4/Pi_HAT_V4_Simple/Pi_HAT_V4_Simple.kicad_pcb (KiCad board)
At the start: 2 copper layers, 71.7 x 71.3 mm, 12 parts, among them J1 MPU 9250, J2 Pi_GPIO, J3 Display, J5 XT60PW-M, J6 Conn_01x04, J7 Conn_01x04, U1 LM2596S

Commit message: Updated lmao
Parts:
- removed J6: Conn_01x04, Connector_PinHeader_2.54mm:PinHeader_1x04_P2.54mm_Vertical
- added G***: LOGO, .pretty:eppl_logo, F.Cu at (90.9, 89.4)
- added TB1: ARDUINO_NANO, .pretty:SHIELD_ARDUINO_NANO, F.Cu at (108.9, 106.9)
- moved S1 45.5 mm to (130.1, 80.7), turned to 0 degrees
- moved J1 45.1 mm to (97.0, 131.4), turned to 180 degrees
- moved J7 13.8 mm to (82.8, 95.9)
- moved J5 2.57 mm to (115.8, 75.5)
Connections:
- J1 pad 1: /3.3V -> /3.3VN
- J1 pad 3: /SCL -> /SCLN
- J1 pad 4: /SDA -> /SDAN
Routing:
- net /SDA: track 172.2 -> 93.6 mm
- net /SCL: track 170.6 -> 96.6 mm
- net GND: track 276.4 -> 211.5 mm
- net /3.3V: track 59.9 -> 17.2 mm
- net /SCLN: track 0.00 -> 36.2 mm
- net /12Vin: track 44.9 -> 11.1 mm
- net /SDAN: track 0.00 -> 26.5 mm
- net /3.3VN: track 0.00 -> 23.4 mm
- net /12Vout: track 136.0 -> 118.4 mm
- net unconnected-(TB1-RESET-Pad28): track 0.00 -> 15.2 mm
Other:
- board size 71.7 x 71.3 mm -> 78.1 x 71.3 mm
- board text added: "BUCK CONVERTER"
- board text added: "NANO"
- board text added: "PI HAT V3 01/24/24 EASY CONTROLS Designed by: Jacob Romeo"
- board text removed: "PI HAT V3 10/21/22 EASY CONTROLS Designed by: Jacob Romeo"
