File: ISAAC/PCB/Pi_HAT/V4/Pi_HAT_V4_Simple/Pi_HAT_V4_Simple.kicad_sch (KiCad schematic)
At the start: 12 parts, among them J1 MPU 9250, J2 Pi_GPIO, J3 Display, J5 XT60PW-M, J6 Conn_01x04, J7 Conn_01x04, U1 LM2596S

Commit message: Updated lmao
Parts:
- removed J6: Conn_01x04, Connector_PinHeader_2.54mm:PinHeader_1x04_P2.54mm_Vertical, symbol Connector_Generic:Conn_01x04
- added TB1: ARDUINO_NANO, .pretty:SHIELD_ARDUINO_NANO, symbol ARDUINO_NANO:ARDUINO_NANO
Connections:
- net 3.3V: no longer J1.1 (Pin_1)
- net GND: now also TB1.29 (COM/GND), TB1.4 (COM/GND)
- net SCL: no longer J1.3 (Pin_3)
- net SDA: no longer J1.4 (Pin_4)
- new net: TB1.28 (RESET), TB1.3 (RESET)
- new net 3.3VN: J1.1 (Pin_1), TB1.17 (3V3)
- new net SCLN: J1.3 (Pin_3), TB1.24 (A5)
- new net SDAN: J1.4 (Pin_4), TB1.23 (A4)
- no-connect marks 40 -> 64
