File: ISAAC/PCB/Pi_HAT/V4/Pi_HAT_V4/Pi_HAT_V4.kicad_sch (KiCad schematic)
At the start: 7 parts, among them J1 MPU 9250, J2 Pi_GPIO, J3 Display

Commit message: updated
Parts:
- added J7: BNO055, Connector_PinHeader_2.54mm:PinHeader_1x06_P2.54mm_Vertical, symbol Connector_Generic:Conn_01x06
Connections:
- net 3.3V: now also J7.1 (Pin_1)
- net GND: now also J7.3 (Pin_3)
- net SCL: now also J7.4 (Pin_4)
- net SDA: now also J7.5 (Pin_5)
- no-connect marks 36 -> 38
Changed lines of the file:
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@@
   (no_connect (at 143.51 83.312))
   (no_connect (at 125.476 80.264))
+  (no_connect (at 143.51 106.934))
+  (no_connect (at 143.51 117.094))
   (no_connect (at 125.476 82.804))
   (no_connect (at 125.476 110.744))
@@
     (stroke (width 0) (type default))
   )
+  (wire (pts (xy 137.16 104.394) (xy 143.51 104.394))
+    (stroke (width 0) (type default))
+  )
   (wire (pts (xy 141.986 57.15) (xy 141.986 56.134))
     (stroke (width 0) (type default))
@@
     (stroke (width 0) (type default))
   )
+  (wire (pts (xy 137.16 114.554) (xy 143.51 114.554))
+    (stroke (width 0) (type default))
+  )
   (wire (pts (xy 183.388 72.898) (xy 187.452 72.898))
+    (stroke (width 0) (type default))
+  )
+  (wire (pts (xy 137.16 112.014) (xy 143.51 112.014))
     (stroke (width 0) (type default))
   )
@@
     (effects (font (size 1.27 1.27)) (justify left bottom))
   )
+  (label "3.3V" (at 137.16 104.394 0) (fields_autoplaced)
+    (effects (font (size 1.27 1.27)) (justify left bottom))
+  )
   (label "3.3V" (at 137.16 73.152 0) (fields_autoplaced)
     (effects (font (size 1.27 1.27)) (justify left bottom))
@@
     (effects (font (size 1.27 1.27)) (justify left bottom))
   )
+  (label "SCL" (at 137.16 112.014 0) (fields_autoplaced)
+    (effects (font (size 1.27 1.27)) (justify left bottom))
+  )
   (label "5V" (at 128.778 62.484 180) (fields_autoplaced)
     (effects (font (size 1.27 1.27)) (justify right bottom))
+  )
+  (label "SDA" (at 137.16 114.554 0) (fields_autoplaced)
+    (effects (font (size 1.27 1.27)) (justify left bottom))
   )
   (symbol (lib_id "Connector_Generic:Conn_02x20_Odd_Even") (at 117.856 85.344 0) (unit 1)
@@
     )
   )
+  (symbol (lib_id "Connector_Generic:Conn_01x06") (at 148.59 109.474 0) (unit 1)
+    (in_bom yes) (on_board yes) (dnp no) (fields_autoplaced)
+    (property "Reference" "J7" (at 151.13 110.109 0)
+      (effects (font (size 1.27 1.27)) (justify left))
+    )
+    (property "Value" "BNO055" (at 151.13 112.649 0)
+      (effects (font (size 1.27 1.27)) (justify left))
+    )
+    (property "Footprint" "Connector_PinHeader_2.54mm:PinHeader_1x06_P2.54mm_Vertical" (at 148.59 109.474 0)
+      (effects (font (size 1.27 1.27)) hide)
+    )
+    (property "Datasheet" "~" (at 148.59 109.474 0)
+      (effects (font (size 1.27 1.27)) hide)
+    )
+    (pin "1")
+    (pin "2")
+    (pin "3")
+    (pin "4")
+    (pin "5")
+    (pin "6")
+    (instances
+      (project "Pi_HAT_V4"
+        (path "/e63e39d7-6ac0-4ffd-8aa3-1841a4541b55"
+          (reference "J7") (unit 1)
+        )
+      )
+    )
+  )
   (symbol (lib_id "Connector_Generic:Conn_01x10") (at 148.59 83.312 0) (unit 1)
     (in_bom yes) (on_board yes) (dnp no) (fields_autoplaced)
@@
         )
       )
+    )
+  )
+  (symbol (lib_id "power:GND") (at 143.51 109.474 270) (unit 1)
+    (in_bom yes) (on_board yes) (dnp no)
+    (property "Reference" "#PWR01" (at 137.16 109.474 0)
+      (effects (font (size 1.27 1.27)) hide)
+    )
+    (property "Value" "GND" (at 140.97 108.204 90)
+      (effects (font (size 1.27 1.27)) (justify right))
+    )
+    (property "Footprint" "" (at 143.51 109.474 0)
+      (effects (font (size 1.27 1.27)) hide)
+    )
+    (property "Datasheet" "" (at 143.51 109.474 0)
+      (effects (font (size 1.27 1.27)) hide)
+    )
+    (pin "1")
+    (instances
+      (project "Pi_HAT_V4"
+        (path "/e63e39d7-6ac0-4ffd-8aa3-1841a4541b55"
+          (reference "#PWR01") (unit 1)
+        )
+      )
